File: Telemetry Hackpad/Hardware/My Telemetry Macropad/Accelerometer.kicad_pcb (KiCad board)
At the start: 2 copper layers, 3.6 x 3.3 mm, 16 parts, among them J1 OLED, J2 MPU 6050, SW1 SW_Push, SW2 SW_Push, SW3 SW_Push, U1 XIAO-RP2040-DIP

Commit message: Added files to repository
Parts:
- removed C1, C2: 0.1uF, Capacitor_SMD:C_0603_1608Metric
- removed C3: 47uF, Capacitor_SMD:C_0603_1608Metric
- removed R1: 330Ω, Resistor_SMD:R_0603_1608Metric
- removed R2, R3: 4.7k, Resistor_SMD:R_0603_1608Metric
- D1, D2, D3, D4: footprint My_Project_Footprints:SK6812MINI-E_fixed (1) -> SK6812MINI-E:SK6812MINI-E_fixed
- moved D3 0.25 mm to (165.0, 135.3)
- moved D2 0.20 mm to (137.0, 95.0), turned to 0 degrees
- turned D4 to 180 degrees
Connections:
- net /SCL renamed SCL
- net /SDA renamed SDA
- net Net-(U1-GPIO26/ADC0/A0) renamed SW1
- net Net-(U1-GPIO27/ADC1/A1) renamed SW2
- net Net-(U1-GPIO28/ADC2/A2) renamed SW3
- D1 pad 1: Net-(D1-DOUT) -> VBUS
- D1 pad 2: /GND -> Net-(D1-DOUT)
- D1 pad 3: Net-(D1-DIN) -> GND
- D1 pad 4: 3V3 -> LEDs
- D2 pad 1: Net-(D2-DOUT) -> VBUS
- D2 pad 2: /GND -> Net-(D2-DOUT)
- D2 pad 3: Net-(D1-DOUT) -> GND
- D2 pad 4: 3V3 -> Net-(D1-DOUT)
- D3 pad 1: Net-(D3-DOUT) -> VBUS
- D3 pad 2: /GND -> Net-(D3-DOUT)
- D3 pad 3: Net-(D2-DOUT) -> GND
- D3 pad 4: 3V3 -> Net-(D2-DOUT)
- D4 pad 1: unconnected-(D4-DOUT-Pad1) -> VBUS
- D4 pad 2: /GND -> unconnected-(D4-DOUT-Pad2)
- D4 pad 3: Net-(D3-DOUT) -> GND
- D4 pad 4: 3V3 -> Net-(D3-DOUT)
- J1 pad 1: 3V3 -> GND
- J1 pad 2: /GND -> +3V3
- J2 pad 1: 3V3 -> +3V3
- J2 pad 2: /GND -> GND
- SW1 pad 1: /GND -> GND
- SW2 pad 1: /GND -> GND
- SW3 pad 1: /GND -> GND
- U1 pad 12: 3V3 -> +3V3
- U1 pad 13: /GND -> GND
- U1 pad 14: unconnected-(U1-VBUS-Pad14) -> VBUS
- U1 pad 4: unconnected-(U1-GPIO29/ADC3/A3-Pad4) -> LEDs
- U1 pad 9: Net-(U1-GPIO2/SCK) -> unconnected-(U1-GPIO2/SCK-Pad9)
Routing:
- net 3V3: track 267.4 -> 0.00 mm, vias 7 -> 0
- net VBUS: track 0.00 -> 230.7 mm
- net /GND: track 199.8 -> 0.00 mm, vias 4 -> 0
- net GND: track 0.00 -> 172.8 mm, vias 0 -> 5
- net +3V3: track 0.00 -> 40.9 mm, vias 0 -> 1
- net LEDs: track 0.00 -> 40.7 mm
- net Net-(D2-DOUT): track 67.6 -> 54.3 mm
- net Net-(U1-GPIO2/SCK): track 11.5 -> 0.00 mm
- net Net-(D1-DOUT): track 69.6 -> 58.7 mm
- net Net-(D3-DOUT): track 64.4 -> 55.7 mm
- net SCL: track 66.4 -> 61.2 mm, vias 2 -> 0
- net Net-(D1-DIN): track 4.77 -> 0.00 mm
- net SDA: track 76.7 -> 72.3 mm, vias 0 -> 1
