File: Telemetry Hackpad/Hardware/My Telemetry Macropad/Accelerometer.kicad_sch (KiCad schematic)
At the start: 15 parts, among them J1 OLED, J2 MPU 6050, SW1 SW_Push, SW2 SW_Push, SW3 SW_Push, U1 XIAO-RP2040-DIP

Commit message: Added files to repository
Parts:
- removed C1, C2: 0.1uF, Capacitor_SMD:C_0603_1608Metric, symbol Device:C
- removed C3: 47uF, Capacitor_SMD:C_0603_1608Metric, symbol Device:C
- removed D1, D2, D3, D4: SK6812MINI-E, My_Project_Footprints:SK6812MINI-E_fixed (1), symbol LED:SK6812MINI
- removed R1, R2: 4.7k, Resistor_SMD:R_0603_1608Metric, symbol Device:R
- added D1, D2, D3, D4: SK6812MINI-E, SK6812MINI-E:SK6812MINI-E_fixed, symbol SK6812MINI-E:SK6812MINI-E
Connections:
- net +3V3: now also J1.2 (VDD); no longer J1.1 (VCC)
- net GND: now also J1.1 (GND), D1.3 (VSS), D2.3 (VSS), D3.3 (VSS), D4.3 (VSS); no longer J1.2 (GND)
- net LEDs: now also D1.4 (DIN)
- net VBUS: now also D1.1 (VDD), D2.1 (VDD), D3.1 (VDD), D4.1 (VDD)
- new net: D2.2 (DOUT), D3.4 (DIN)
- new net: D1.2 (DOUT), D2.4 (DIN)
- new net: D3.2 (DOUT), D4.4 (DIN)
